Commit message: Add fingers macro, modified joints from revolute to fixed

File: robotiq_3f_gripper_visualization/cfg/robotiq_hand_macro.urdf.xacro (robot description, xacro)
@@ -7,12 +7,13 @@
 -->
 <robot xmlns:xacro="http://www.ros.org/wiki/xacro" name="robotiq_hand">
-  <xacro:macro name="robotiq_finger" params="prefix">
-    <!-- Link list -->
-    <!-- Link 0 -->
-    <link name="${prefix}link_0">
+  <!-- Include fingers -->
+  <xacro:include filename="$(find robotiq_3f_gripper_visualization)/cfg/robotiq_finger.urdf.xacro" />
+  <xacro:macro name="robotiq_hand" params="prefix *origin reflect parent">
+    <!-- link list -->
+    <!-- Link palm -->
+    <link name="${prefix}palm">
       <visual>
-        <origin xyz="0 0 0" rpy="0 0 0"/>
         <geometry>
-          <mesh filename="package://robotiq_3f_gripper_visualization/meshes/robotiq-3f-gripper_articulated/visual/link_0.dae" />
+          <mesh filename="package://robotiq_3f_gripper_visualization/meshes/robotiq-3f-gripper_articulated/visual/palm.dae" />
         </geometry>
         <material name="green">
@@ -23,5 +24,5 @@
         <origin rpy="0 0 0" xyz="0 0 0"/>
         <geometry>
-          <mesh filename="package://robotiq_3f_gripper_visualization/meshes/robotiq-3f-gripper_articulated/collision/link_0.STL" />
+          <box size="0.1 0.1 0.1"/>
         </geometry>
         <material name="yellow">
@@ -30,607 +31,14 @@
       </collision>
       <inertial>
-        <mass value="0.1"/>
-        <origin xyz="-0.01 0 0"/>
-        <inertia ixx="0.000018" ixy="0" ixz="0" iyy="0.000025" iyz="0" izz="0.000025"/>
+        <origin rpy="0 0 0" xyz="0 0 0"/>
+        <mass value="1.3"/>
+        <inertia ixx="0.0035" ixy="0" ixz="-0" iyy="0.0035" iyz="0" izz="0.0035"/>
       </inertial>
     </link>
-    <gazebo reference="${prefix}link_0">
-      <mu1>1.1</mu1>
-      <mu2>1.1</mu2>
-    </gazebo>
-    <!-- Link 1 -->
-    <link name="${prefix}link_1">
-      <visual>
-        <origin rpy="0 0 ${3.1416/2}" xyz="0 0.05717 0"/>
-        <geometry>
-          <mesh filename="package://robotiq_3f_gripper_visualization/meshes/robotiq-3f-gripper_articulated/visual/link_1.dae" />
-        </geometry>
-        <material name="green"/>
-      </visual>
-      <collision>
-        <origin rpy="0 0 ${3.1416/2}" xyz="0 0.05717 0"/>
-        <geometry>
-          <mesh filename="package://robotiq_3f_gripper_visualization/meshes/robotiq-3f-gripper_articulated/collision/link_1.STL"/>
-        </geometry>
-        <material name="yellow">
-          <color rgba="0 1 1 1"/>
-        </material>
-      </collision>
-      <inertial>
-        <origin rpy="0 0 ${3.1416/2}" xyz="0.00053 0.03218 0"/>
-        <mass value="0.047"/>
-        <inertia ixx= "0.00000499332"
-                 ixy= "0.00000091312"
-                 ixz="-0.00000000120"
-                 iyy= "0.00006434531"
-                 iyz="-0.00000000007"
-                 izz= "0.00006061917"/>
-      </inertial>
-    </link>
-    <gazebo reference="${prefix}link_1">
-      <mu1>1.1</mu1>
-      <mu2>1.1</mu2>
-    </gazebo>
-    <!-- Link 2 -->
-    <link name="${prefix}link_2">
-      <visual>
-        <origin rpy="0 0 ${3.1416/2}" xyz="0 0.03810 0.0075"/>
-        <geometry>
-          <mesh filename="package://robotiq_3f_gripper_visualization/meshes/robotiq-3f-gripper_articulated/visual/link_2.dae" />
-        </geometry>
-        <material name="green"/>
-      </visual>
-      <collision>
-        <origin rpy="0 0 ${3.1416/2}" xyz="0 0.03810 0.0075"/>
-          <geometry>
-            <mesh filename="package://robotiq_3f_gripper_visualization/meshes/robotiq-3f-gripper_articulated/collision/link_2.STL"/>
-          </geometry>
-        <material name="yellow"/>
-      </collision>
-      <inertial>
-        <origin rpy="0 0 ${3.1416/2}" xyz="0.00048 0.02167 0.00018"/>
-        <mass value="0.03284"/>
-        <inertia ixx="0.00000348008"
-                 ixy="0.00000031940"
-                 ixz="0.00000013041"
-                 iyy="0.00002248123"
-                 iyz="0.00000000291"
-                 izz="0.00001986346"/>
-      </inertial>
-    </link>
-    <gazebo reference="${prefix}link_2">
-      <mu1>1.1</mu1>
-      <mu2>1.1</mu2>
-    </gazebo>
-    <!-- Link 3 -->
-    <link name="${prefix}link_3">
-      <visual>
-        <origin xyz="0 0 0" rpy="0 0 0"/>
-        <geometry>
-          <mesh filename="package://robotiq_3f_gripper_visualization/meshes/robotiq-3f-gripper_articulated/visual/link_3.dae" />
-        </geometry>
-        <material name="green"/>
-      </visual>
-      <collision>
-        <origin xyz="0 0 0" rpy="0 0 0"/>
-        <geometry>
-          <mesh filename="package://robotiq_3f_gripper_visualization/meshes/robotiq-3f-gripper_articulated/collision/link_3.STL"/>
-        </geometry>
-        <material name="yellow"/>
-      </collision>
-      <inertial>
-        <origin rpy="0 0 0" xyz="0.01626 0.00049 0.0002"/>
-        <mass value="0.03354"/>
-        <inertia ixx="0.00000305151"
-                 ixy="0.00000089792"
-                 ixz="0.00000000249"
-                 iyy="0.00001427978"
-                 iyz="-0.00000001191"
-                 izz="0.00001264126"/>
-      </inertial>
-    </link>
-    <gazebo reference="${prefix}link_3">
-      <mu1>1.1</mu1>
-      <mu2>1.1</mu2>
-    </gazebo>
-    <!-- Link proximal actuating hinge -->
-    <link name="${prefix}link_proximal_actuating_hinge">
-      <visual>
-        <origin rpy="0 0 0" xyz="0.01429 0 0"/>
-        <geometry>
-          <box size="0.02858 .0075 .002"/>
-        </geometry>
-      </visual>
-      <collision>
-        <origin rpy="0 0 0" xyz="0.01429 0 0"/>
-         <geometry>
-          <box size="0.02858 .0075 .002"/>
-        </geometry>
-      </collision>
-      <inertial>
-        <origin rpy="0 0 0" xyz="0.0012 -0.00162 -0.00161"/>
-        <mass value="0.02647"/>
-        <inertia ixx= "0.00000156447"
-                 ixy= "0.000000236226"
-                 ixz="-0.00000014862"
-                 iyy= "0.00000221068"
-                 iyz="-0.00000014369"
-                 izz= "0.00000323175"/>
-      </inertial>
-    </link>
-    <gazebo reference="${prefix}link_proximal_actuating_hinge">
-      <mu1>1.1</mu1>
-      <mu2>1.1</mu2>
-    </gazebo>
-    <!-- Link paraproximal actuating hinge -->
-    <link name="${prefix}link_paraproximal_actuating_hinge">
-      <visual>
-        <origin rpy="0 0 0" xyz="0.01143 0 0"/>
-        <geometry>
-          <box size="0.02286 .0075 .002"/>
-        </geometry>
-      </visual>
-      <collision>
-        <origin rpy="0 0 0" xyz="0.01143 0 0"/>
-         <geometry>
-          <box size="0.02286 .0075 .002"/>
-        </geometry>
-      </collision>
-      <inertial>
-        <origin rpy="0 0 0" xyz="0.0064 0 0"/>
-        <!-- copied from proximal_actuating_hinge -->
-        <mass value="0.00362"/>
-        <inertia ixx= "0.00000012043"
-                 ixy= "0"
-                 ixz= "0"
-                 iyy= "0.00000053588"
-                 iyz= "0"
-                 izz= "0.00000065322"/>
-      </inertial>
-    </link>
-    <gazebo reference="${prefix}link_paraproximal_actuating_hinge">
-      <mu1>1.1</mu1>
-      <mu2>1.1</mu2>
-    </gazebo>
-    <!-- Link proximal actuating bar -->
-    <link name="${prefix}link_proximal_actuating_bar">
-      <visual>
-        <origin rpy="0 0 0" xyz="0.026789 0 0"/>
-        <geometry>
-          <box size="0.05398 .0075 .002"/>
-        </geometry>
-      </visual>
-      <collision>
-        <origin rpy="0 0 0" xyz="0.026789 0 0"/>
-         <geometry>
-          <box size="0.05398 .0075 .002"/>
-        </geometry>
-      </collision>
-      <inertial>
-        <origin rpy="0 0 0" xyz="0.02699 -0.00122 0"/>
-        <mass value="0.00659"/>
-        <inertia ixx= "0.00000008348"
-                 ixy="-0.0000002179"
-                 ixz= "0.00000000134"
-                 iyy= "0.00000719076"
-                 iyz= "0"
-                 izz= "0.00000718272"/>
-      </inertial>
-    </link>
-    <gazebo reference="${prefix}link_proximal_actuating_bar">
-      <mu1>1.1</mu1>
-      <mu2>1.1</mu2>
-    </gazebo>
-    <!-- Link paraproximal bar -->
-    <link name="${prefix}link_paraproximal_bar">
-      <visual>
-        <origin rpy="0 0 0" xyz="0.02885 0 0"/>
-        <geometry>
-          <box size="0.05770 .0075 .002"/>
-        </geometry>
-      </visual>
-      <collision>
-        <origin rpy="0 0 0" xyz="0.02885 0 0"/>
-         <geometry>
-          <box size="0.05770 .0075 .002"/>
-        </geometry>
-      </collision>
-      <inertial>
-        <origin rpy="0 0 0" xyz="0.02858 -0.00129 0"/>
-        <mass value="0.00732"/>
-        <inertia ixx= "0.00000009065"
-                 ixy="-0.00000027047"
-                 ixz= "0.00000000142"
-                 iyy= "0.00000878034"
-                 iyz= "0"
-                 izz= "0.00000877558"/>
-      </inertial>
-    </link>
-    <gazebo reference="${prefix}link_paraproximal_bar">
-      <mu1>1.1</mu1>
-      <mu2>1.1</mu2>
-    </gazebo>
-    <!-- Link median actuating hinge -->
-    <link name="${prefix}link_median_actuating_hinge">
-      <visual>
-        <origin rpy="0 0 0" xyz="0 0 0"/>
-        <geometry>
-          <box size=".02 .02 .002"/>
-        </geometry>
-      </visual>
-      <collision>
-        <origin rpy="0 0 0" xyz="0 0 0"/>
-         <geometry>
-          <box size=".02 .02 .002"/>
-        </geometry>
-      </collision>
-      <inertial>
-        <origin rpy="0 0 0" xyz="0.0092 0.00514 0"/>
-        <mass value="0.00359"/>
-        <inertia ixx= "0.00000024735"
-                 ixy= "0.00000023619"
-                 ixz= "0"
-                 iyy= "0.00000047681"
-                 iyz= "0"
-                 izz= "0.00000071813"/>
-      </inertial>
-    </link>
-    <gazebo reference="${prefix}link_median_actuating_hinge">
-      <mu1>1.1</mu1>
-      <mu2>1.1</mu2>
-    </gazebo>
-    <!-- Link median bar -->
-    <link name="${prefix}link_median_bar">
-      <visual>
-        <origin rpy="0 0 0" xyz="0.01905 0 0"/>
-        <geometry>
-          <box size="0.0381 .0075 .002"/>
-        </geometry>
-      </visual>
-      <collision>
-        <origin rpy="0 0 0" xyz="0.01905 0 0"/>
-         <geometry>
-          <box size="0.0381 .0075 .002"/>
-        </geometry>
-      </collision>
-      <inertial>
-        <origin rpy="0 0 0" xyz="0.01905 -0.00107 0"/>
-        <mass value="0.00538"/>
-        <inertia ixx= "0.00000006639"
-                 ixy="-0.00000010996"
-                 ixz= "0.00000000094"
-                 iyy= "0.00000305318"
-                 iyz= "0"
-                 izz= "0.00000304657"/>
-      </inertial>
-    </link>
-    <gazebo reference="${prefix}link_median_bar">
-      <mu1>1.1</mu1>
-      <mu2>1.1</mu2>
-    </gazebo>
-    <!-- Link paramedian hinge -->
-    <link name="${prefix}link_paramedian_hinge">
-      <visual>
-        <origin rpy="0 0 0" xyz="0 0 0"/>
-        <geometry>
-          <box size=".02 .02 .002"/>
-        </geometry>
-      </visual>
-      <collision>
-        <origin rpy="0 0 0" xyz="0 0 0"/>
-         <geometry>
-          <box size=".02 .02 .002"/>
-        </geometry>
-      </collision>
-      <inertial>
-        <origin rpy="0 0 0" xyz="-0.01025 0.00046 0"/>
-        <mass value="0.00276"/>
-        <inertia ixx= "0.00000004213"
-                 ixy="-0.00000001491"
-                 ixz= "0"
-                 iyy= "0.00000050258"
-                 iyz= "0"
-                 izz= "0.00000054007"/>
-      </inertial>
-    </link>
-    <gazebo reference="${prefix}link_paramedian_hinge">
-      <mu1>1.1</mu1>
-      <mu2>1.1</mu2>
-    </gazebo>
-    <!-- Link median bar underactuated -->
-    <link name="${prefix}link_median_bar_underactuated">
-      <visual>
-        <origin rpy="0 0 0" xyz="0.01905 0 0"/>
-        <geometry>
-          <box size="0.0381 .0075 .002"/>
-        </geometry>
-      </visual>
-      <collision>
-        <origin rpy="0 0 0" xyz="0.01905 0 0"/>
-         <geometry>
-          <box size="0.0381 .0075 .002"/>
-        </geometry>
-      </collision>
-      <inertial>
-        <origin rpy="0 0 0" xyz="0.01905 -0.00107 0"/>
-        <mass value="0.00538"/>
-        <inertia ixx= "0.00000006639"
-                 ixy="-0.00000010996"
-                 ixz="-0.00000000094"
-                 iyy= "0.00000305318"
-                 iyz= "0"
-                 izz= "0.00000304657"/>
-      </inertial>
-    </link>
-    <gazebo reference="${prefix}link_median_bar_underactuated">
-      <mu1>1.1</mu1>
-      <mu2>1.1</mu2>
-    </gazebo>
-    <!-- Link paradistal hinge -->
-    <link name="${prefix}link_paradistal_hinge">
-      <visual>
-        <origin rpy="0 0 0" xyz="0 0 0"/>
-        <geometry>
-          <box size=".02 .02 .002"/>
-        </geometry>
-      </visual>
-      <collision>
-        <origin rpy="0 0 0" xyz="0 0 0"/>
-         <geometry>
-          <box size=".02 0.02 .002"/>
-        </geometry>
-      </collision>
-      <inertial>
-        <origin rpy="0 0 0" xyz="0.00548 0 0"/>
-        <mass value="0.00158"/>
-        <inertia ixx= "0.00000001907"
-                 ixy= "0"
-                 ixz= "0"
-                 iyy= "0.00000010970"
-                 iyz= "0"
-                 izz= "0.00000012610"/>
-      </inertial>
-    </link>
-    <gazebo reference="${prefix}link_paradistal_hinge">
+    <gazebo reference="${prefix}palm">
       <mu1>1.1</mu1>
       <mu2>1.1</mu2>
     </gazebo>
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